Commit message: [add] add IMU sensor

File: omnibot3_description/robot/omnibot3.urdf.xacro (robot description, xacro)
@@ -3,4 +3,5 @@
   <xacro:include filename="$(find omnibot3_description)/urdf/base/base.urdf.xacro"/>
   <xacro:include filename="$(find omnibot3_description)/urdf/wheel/wheel.urdf.xacro"/>
+  <xacro:include filename="$(find omnibot3_description)/urdf/sensors/imu/imu.urdf.xacro"/>
   <!-- =============== Link & Joint =============== -->
   <!-- Base -->
@@ -22,4 +23,9 @@
     <origin rpy="0 0 ${7*M_PI/6}" xyz="${0.07*cos(M_PI/6)*cos(5*M_PI/3)} ${-0.07*cos(5*M_PI/6)*sin(5*M_PI/3)} 0.025"/>
   </xacro:wheel>
+  <!-- Sensors -->
+  <!-- IMU -->
+  <xacro:imu id_num="1" parent="base_link">
+    <origin xyz="0.05 0 0.052" rpy="0 0 0"/>
+  </xacro:imu>
   <!-- =============== Transmission =============== -->
   <xacro:wheel_trans id_num="1"/>
@@ -38,3 +44,5 @@
   <xacro:wheel_gazebo id_num="2"/>
   <xacro:wheel_gazebo id_num="3"/>
+  <!-- IMU -->
+  <xacro:imu_gazebo id_num="1"/>
 </robot>

File: omnibot3_description/urdf/common.xacro (robot description, xacro)
@@ -6,5 +6,6 @@
     <inertia ixx="${((radius*radius)/4 + (length*length)/12)*mass}" ixy="0" ixz="0" iyy="${((radius*radius)/4 + (length*length)/12)*mass}" iyz="0" izz="${(mass*radius*radius)/2}"/>
   </xacro:macro>
-  <xacro:macro name="box_inertial" param="mass height width depth">
+  <xacro:macro name="box_inertial" params="mass height width depth">
+    <mass value="${mass}"/>
     <inertia ixx="${(mass*(width*width+depth*depth))/12}" ixy="0" ixz="0" iyy="${(mass*(height*height+depth*depth))/12}" iyz="0" izz="${(mass*(height*height+width*width))/12}"/>
   </xacro:macro>
